File: pcb2/tomo.kicad_pcb (KiCad board)
At the start: 2 copper layers, 108.8 x 75.7 mm, 18 parts, among them U1 BluePill_STM32F103C, U2 4051, U3 4051

Commit message: tes ok
Connections:
- U1 pad 30: /L_C -> /L_A
- U1 pad 32: /L_A -> /L_C
- U2 pad 11: /L_C -> /L_A
- U2 pad 9: /L_A -> /L_C
Routing:
- net /L_C: track 49.7 -> 36.3 mm
- net /L_A: track 36.3 -> 49.7 mm
Changed lines of the file:
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@@
   (general
     (links 61)
-    (no_connects 18)
+    (no_connects 0)
     (area 41.749999 20.749999 151.050001 96.950001)
     (thickness 1.6)
@@
   )
   (setup
-    (last_trace_width 1)
+    (last_trace_width 0.25)
     (user_trace_width 0.6)
     (user_trace_width 0.8)
@@
       (net 27 "Net-(U1-Pad29)"))
     (pad 30 thru_hole oval (at 15.24 25.3492 90) (size 1.7272 2.25) (drill 1.016) (layers *.Cu *.Mask F.SilkS)
-      (net 33 /L_C))
+      (net 31 /L_A))
     (pad 31 thru_hole oval (at 15.24 22.8092 90) (size 1.7272 2.25) (drill 1.016) (layers *.Cu *.Mask F.SilkS)
       (net 32 /L_B))
     (pad 32 thru_hole oval (at 15.24 20.2692 90) (size 1.7272 2.25) (drill 1.016) (layers *.Cu *.Mask F.SilkS)
-      (net 31 /L_A))
+      (net 33 /L_C))
     (pad 33 thru_hole oval (at 15.24 17.7292 90) (size 1.7272 2.25) (drill 1.016) (layers *.Cu *.Mask F.SilkS)
       (net 34 /L_INH))
@@
       (net 42 /L7))
     (pad 9 thru_hole oval (at 7.62 17.78) (size 1.6 1.6) (drill 0.8) (layers *.Cu *.Mask)
-      (net 31 /L_A))
+      (net 33 /L_C))
     (pad 2 thru_hole oval (at 0 2.54) (size 1.6 1.6) (drill 0.8) (layers *.Cu *.Mask)
       (net 41 /L6))
@@
       (net 9 "Net-(R-LED5-Pad2)"))
     (pad 11 thru_hole oval (at 7.62 12.7) (size 1.6 1.6) (drill 0.8) (layers *.Cu *.Mask)
-      (net 33 /L_C))
+      (net 31 /L_A))
     (pad 4 thru_hole oval (at 0 7.62) (size 1.6 1.6) (drill 0.8) (layers *.Cu *.Mask)
       (net 40 /L5))
@@
   (segment (start 131.975 50.8) (end 128.2 50.8) (width 0.8) (layer B.Cu) (net 9))
   (segment (start 128.2 50.8) (end 128.055 50.945) (width 0.8) (layer B.Cu) (net 9))
-  (segment (start 127.1 66.6) (end 132.72 66.6) (width 0.8) (layer B.Cu) (net 31))
-  (segment (start 132.72 66.6) (end 135.675 63.645) (width 0.8) (layer B.Cu) (net 31))
-  (segment (start 125.6 65.1) (end 127.1 66.6) (width 0.8) (layer B.Cu) (net 31))
-  (segment (start 125.6 62.2) (end 125.6 65.1) (width 0.8) (layer B.Cu) (net 31))
-  (segment (start 124.5728 61.1728) (end 125.6 62.2) (width 0.8) (layer B.Cu) (net 31))
-  (segment (start 104.5411 61.1728) (end 124.5728 61.1728) (width 0.8) (layer B.Cu) (net 31))
+  (segment (start 104.5411 66.2528) (end 106.4661 66.2528) (width 0.8) (layer B.Cu) (net 31))
+  (segment (start 140 60.2) (end 138.3 58.5) (width 0.8) (layer B.Cu) (net 31))
+  (segment (start 106.4661 66.2528) (end 106.5133 66.3) (width 0.8) (layer B.Cu) (net 31))
+  (segment (start 106.5133 66.3) (end 122 66.3) (width 0.8) (layer B.Cu) (net 31))
+  (segment (start 122 66.3) (end 125.6 69.9) (width 0.8) (layer B.Cu) (net 31))
+  (segment (start 125.6 69.9) (end 136.5 69.9) (width 0.8) (layer B.Cu) (net 31))
+  (segment (start 138.3 58.5) (end 138.235 58.565) (width 0.8) (layer B.Cu) (net 31))
+  (segment (start 136.5 69.9) (end 140 66.4) (width 0.8) (layer B.Cu) (net 31))
+  (segment (start 138.235 58.565) (end 135.675 58.565) (width 0.8) (layer B.Cu) (net 31))
+  (segment (start 140 66.4) (end 140 60.2) (width 0.8) (layer B.Cu) (net 31))
   (segment (start 104.5411 63.7128) (end 106.4661 63.7128) (width 0.8) (layer B.Cu) (net 32))
   (segment (start 123.1 63.7) (end 123.7 64.3) (width 0.8) (layer B.Cu) (net 32))
@@
   (segment (start 135.5 68.2) (end 138.4 65.3) (width 0.8) (layer B.Cu) (net 32))
   (segment (start 138.4 62) (end 137.505 61.105) (width 0.8) (layer B.Cu) (net 32))
-  (segment (start 104.5411 66.2528) (end 106.4661 66.2528) (width 0.8) (layer B.Cu) (net 33))
-  (segment (start 140 60.2) (end 138.3 58.5) (width 0.8) (layer B.Cu) (net 33))
-  (segment (start 106.4661 66.2528) (end 106.5133 66.3) (width 0.8) (layer B.Cu) (net 33))
-  (segment (start 106.5133 66.3) (end 122 66.3) (width 0.8) (layer B.Cu) (net 33))
-  (segment (start 122 66.3) (end 125.6 69.9) (width 0.8) (layer B.Cu) (net 33))
-  (segment (start 125.6 69.9) (end 136.5 69.9) (width 0.8) (layer B.Cu) (net 33))
-  (segment (start 138.3 58.5) (end 138.235 58.565) (width 0.8) (layer B.Cu) (net 33))
-  (segment (start 136.5 69.9) (end 140 66.4) (width 0.8) (layer B.Cu) (net 33))
-  (segment (start 138.235 58.565) (end 135.675 58.565) (width 0.8) (layer B.Cu) (net 33))
-  (segment (start 140 66.4) (end 140 60.2) (width 0.8) (layer B.Cu) (net 33))
+  (segment (start 127.1 66.6) (end 132.72 66.6) (width 0.8) (layer B.Cu) (net 33))
+  (segment (start 132.72 66.6) (end 135.675 63.645) (width 0.8) (layer B.Cu) (net 33))
+  (segment (start 125.6 65.1) (end 127.1 66.6) (width 0.8) (layer B.Cu) (net 33))
+  (segment (start 125.6 62.2) (end 125.6 65.1) (width 0.8) (layer B.Cu) (net 33))
+  (segment (start 124.5728 61.1728) (end 125.6 62.2) (width 0.8) (layer B.Cu) (net 33))
+  (segment (start 104.5411 61.1728) (end 124.5728 61.1728) (width 0.8) (layer B.Cu) (net 33))
   (segment (start 104.5411 58.6328) (end 127.9872 58.6328) (width 0.8) (layer B.Cu) (net 34))
   (segment (start 127.9872 58.6328) (end 128.055 58.565) (width 0.8) (layer B.Cu) (net 34))
